File: kicad/haven_dev_board.kicad_sch (KiCad schematic)
At the start: 89 parts, among them CN1 BM46B-12DS-0.35V(51), J1 CLE-107-01-G-DV, Q1 CSD23382F4, Q2 CSD13380F3T, Q3 CSD13380F3T, SW1 TS2819A 230GF, U1 BMX160, U10 SN74AXC4T774RSVR, U12 GT-USB-9047A, U13 SPH0641LU4H-1, U14 MX25R6435FBFIL0, U15 ADAU1860BCBZRL, U2 BQ25120AYFPR, U3 AP22916BCA4-7, U4 XL-0201SURC, U5 KTD2026, U6 BQ27220YZFR, U8 1MΩ, U9 AP22916BCA4-7, X1 Q13FC1350000200

Commit message: Fix U1 part label: BMX160 -> BMI160 (no magnetometer on this board)
The schematic's Value property said BMX160 (Bosch 9-axis IMU, has an
on-die magnetometer) while the sourced Manufacturer Part in the BOM was
BMI160 (6-axis, no magnetometer) -- a real mismatch flagged earlier as
unresolved, since both packages/pinouts are identical and don't
disambiguate on their own.

Resolved by checking the actual wiring: U1 pins 2/3 (ASDX/ASCX, BMI160's
external-magnetometer aux interface) are tied to GND, which is BMI160's
own documented "aux interface unused" reference pattern. BMX160 has no
equivalent external aux-mag pins to ground -- its magnetometer is on-die
using that interface internally -- so this wiring is specifically valid
for BMI160, not BMX160.

Corrected the schematic's U1 Value to BMI160 and updated the BOM note
from "discrepancy" to "resolved." No functional change: nothing in
Haven's firmware uses IMU/magnetometer data today.
Parts:
- U1: value BMX160 -> BMI160
Changed lines of the file:
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@@
   (symbol (lib_id "haven_dev_board:U1") (at 210.820 193.040 0) (unit 1)
     (property "Reference" "U1" (at 210.820 188.040 0) (effects (font (size 1.27 1.27))))
-    (property "Value" "BMX160" (at 210.820 198.040 0) (effects (font (size 1.27 1.27))))
+    (property "Value" "BMI160" (at 210.820 198.040 0) (effects (font (size 1.27 1.27))))
   )
   (label "GND" (at 198.120 200.660 0) (effects (font (size 1.27 1.27)) (justify left)))
