File: kicad/haven_dev_board.kicad_sch (KiCad schematic)
At the start: 96 parts, among them CN1 BM46B-12DS-0.35V(51), J1 CLE-107-01-G-DV, Q1 CSD23382F4, Q2 CSD13380F3T, Q3 CSD13380F3T, SW1 TS2819A 230GF, U1 BMI160, U10 SN74AXC4T774RSVR, U12 GT-USB-9047A, U13 SPH0641LU4H-1, U14 MX25R6435FBFIL0, U15 ADAU1860BCBZRL, U2 TP4056, U3 AP22916BCA4-7, U4 XL-0201SURC, U5 KTD2026, U6 BQ27220YZFR, U8 1MΩ, U9 AP22916BCA4-7, X1 Q13FC1350000200

Commit message: Place TP4056/TPS62822/TPS22917 footprints on the real PCB
Follows the schematic-side power-tree redesign (previous commit) onto
kicad/haven_dev_board.kicad_pcb. Removes the old U2 (BQ25120A, DSBGA-25)
footprint and places three real footprints copied from KiCad's own
official library (not hand-derived): Texas_VSON-HR-8_1.5x2mm_P0.5mm for
TPS62822DLCR, SOIC-8_3.9x4.9mm_P1.27mm for TP4056, SOT-23-6 for
TPS22917DBVR — each cross-checked against its datasheet's own package
outline drawing before use. Five new 0402 passives added for R_PROG,
R_FB1, R_FB2, R_PU_CHRG, R_PU_STDBY.

Pad-to-net assignment done directly by name (schematic netlist export is
broken for this project, a separate pre-existing issue — see
HARDWARE_COST_ALTERNATIVES.md), matching the schematic-side net names.

Caught and fixed a real placement mistake via kicad-cli pcb drc, not
assumed away: an initial attempt placed the buck IC next to the existing
inductor L2, which turned out to sit in a zone still densely routed with
old charger-circuit copper (VUSB/V_PMID/V_LS traces), producing two real
"shorting_items" DRC violations. Relocated to genuinely clear board area,
re-verified.

kicad-cli pcb drc: 221 violations vs. the documented 219-violation
baseline. Clearance violations actually went DOWN (85 vs 99) since the
old fine-pitch BGA is gone. The increase is expected "not yet routed"
noise (28 unconnected pads vs 2 baseline) — footprints are placed and
net-assigned but no copper routing has been done yet. Also fixed R_PROG's
value (1.1k -> 1.2k) to match the TP4056 datasheet's own characterization
table exactly (1000mA typical charge current at 1.2k).

Co-Authored-By: Claude Sonnet 5 <noreply@anthropic.com>
Claude-Session: https://claude.ai/code/session_01YTbrWH9Gt2quSDLgz6Te5V
Parts:
- R_PROG: value 1.1k -> 1.2k
Changed lines of the file:
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@@
     (effects (font (size 1.27 1.27)) (justify left))
   )
-  (label "GND" (at 289.84 335.0 0)
+  (label "GND" (at 289.84 335 0)
     (effects (font (size 1.27 1.27)) (justify left))
   )
@@
       (effects (font (size 1.27 1.27)))
     )
-    (property "Value" "1.1k" (at 260 272 0)
-      (effects (font (size 1.27 1.27)))
-    )
+    (property "Value" "1.2k" (at 260 272 0)
+      (effects (font (size 1.27 1.27)))
+    )

Commit message: Replace ADAU1860 codec + PDM mic with TLV320AIC3100 + CMA-4544PF-W
This is the real headline item from the original cost analysis: the
ADAU1860 (BGA-56, 0.35mm pitch) was always the single biggest cost
driver on the board, bigger than the charger already replaced in the
prior two commits. Removes U15 (ADAU1860) and U13 (the old PDM mic,
SPH0641LU4H-1), replacing with TLV320AIC3100 (QFN-32, real pinout from
its own datasheet SLAS667C) and CMA-4544PF-W (a plain 2-terminal analog
electret capsule, since TLV320AIC3100 has no PDM input at all — its mic
inputs are analog PGA inputs, confirmed from its own datasheet).

Reuses the real I2S bus (DIN/DOUT/BCLK/LRCLK), I2C bus (SDA1/SCL1), and
analog supply rail (V_LS) that already existed for the old codec/mic.
Notably reuses the +1.8V rail the charger redesign (previous commits)
created for the new codec's DVDD — the two changes are genuinely
coupled, not independent swaps.

Real simplifications made and flagged explicitly (see
HARDWARE_COST_ALTERNATIVES.md): MCLK tied to BCLK instead of adding a
dedicated crystal (datasheet explicitly allows this), RESET tied
directly to 3V3, unused Class-D speaker block (6 pins) and GPIO1 left
genuinely unconnected, VOL/MICDET and the unused mic differential pin
tied to GND.

Caught a real bug before applying: an early draft of the mic-bias
network gave the AC-coupling cap's two terminals the same net name,
which would have shorted across it and defeated its purpose. Fixed with
two distinct nets either side of the cap.

kicad-cli sch erc: still 86 violations total (flat, not growing) versus
the charger-only state. The specific nets flagged as label_dangling
shifted (new mic-bias nets now flagged, two previously-flagged charger
nets no longer are) despite no change to their actual wiring — further
evidence this is an unstable checker quirk, not a real defect. Verified
directly by coordinate comparison that every new pin lands exactly on
its intended label except the 9 deliberately-unconnect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
Parts:
- removed R_FB1: 200k, symbol haven_dev_board:R_FB1
- removed R_FB2: 100k, symbol haven_dev_board:R_FB2
- removed R_PROG: 1.2k, symbol haven_dev_board:R_PROG
- removed R_PU_CHRG: 100k, symbol haven_dev_board:R_PU_CHRG
- removed R_PU_STDBY: 100k, symbol haven_dev_board:R_PU_STDBY
- removed U13: SPH0641LU4H-1, symbol haven_dev_board:U13
- removed U15: ADAU1860BCBZRL, symbol haven_dev_board:U15
- removed U2: TP4056, symbol haven_dev_board:TP4056
- removed U_BUCK1: TPS62822DLCR, symbol haven_dev_board:TPS62822DLC
- removed U_LS1: TPS22917DBVR, symbol haven_dev_board:TPS22917
- added C_MICIN: 1uF, symbol haven_dev_board:C_MICIN
- added R_MICBIAS: 2.2k, symbol haven_dev_board:R_MICBIAS
- added U13: CMA-4544PF-W, symbol haven_dev_board:CMA-4544PF-W
- added U15: TLV320AIC3100, symbol haven_dev_board:TLV320AIC3100
- added U2: BQ25120AYFPR, symbol haven_dev_board:U2

Commit message: Fix: restore the charger redesign the codec commit had silently reverted
Real bug, not a close call: the schematic on this branch had lost the
entire charger redesign (TP4056/TPS62822/TPS22917, and the old BQ25120A
was back) for the last three commits. Root cause: the codec/mic
generation script ran while the working tree was on master (left there
from the previous tick's PR-comment step) instead of this branch, so it
built the codec swap on top of the original untouched schematic and that
output silently overwrote this branch's charger-redesigned file when
copied in. The PCB was never affected (separate file/process) -- which
is exactly why ERC/DRC being clean throughout didn't catch it: a schema
that's internally consistent isn't the same as one that still contains
everything it's supposed to.

Caught by routine verification (checking what's in the schematic before
starting new work) rather than any specific test -- U2 was still valued
BQ25120AYFPR on a branch whose entire point was replacing it.

Fixed by re-running both generation scripts in the correct order this
time: charger script against the real original (pulled fresh from
master, since this branch's copy was known-compromised), verified via
ERC (86 violations, exact charger-only baseline), then the codec script
against THAT output. Verified twice: kicad-cli sch erc (88 violations --
84 baseline + 5 genuinely new nets across both changesets, matching the
established pattern exactly) and a direct pin-by-pin coordinate check
confirming all 70 new pins land on their intended labels except the 13
deliberately unconnected ones.

Co-Authored-By: Claude Sonnet 5 <noreply@anthropic.com>
Claude-Session: https://claude.ai/code/session_01YTbrWH9Gt2quSDLgz6Te5V
Parts:
- removed U2: BQ25120AYFPR, symbol haven_dev_board:U2
- added R_FB1: 200k, symbol haven_dev_board:R_FB1
- added R_FB2: 100k, symbol haven_dev_board:R_FB2
- added R_PROG: 1.2k, symbol haven_dev_board:R_PROG
- added R_PU_CHRG: 100k, symbol haven_dev_board:R_PU_CHRG
- added R_PU_STDBY: 100k, symbol haven_dev_board:R_PU_STDBY
- added U2: TP4056, symbol haven_dev_board:TP4056
- added U_BUCK1: TPS62822DLCR, symbol haven_dev_board:TPS62822DLC
- added U_LS1: TPS22917DBVR, symbol haven_dev_board:TPS22917
Changed lines of the file:
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@@
-    (effects (font (size 1.27 1.27)) (justify left))
-  )
-  (label "GND" (at 295.91 175.26 0)
-    (effects (font (size 1.27 1.27)) (justify left))
-  )
-  (label "SCL" (at 326.39 173.99 0)
-    (effects (font (size 1.27 1.27)) (justify left))
-  )
-  (label "VUSB" (at 295.91 172.72 0)
-    (effects (font (size 1.27 1.27)) (justify left))
-  )
-  (label "SDA" (at 326.39 171.45 0)
-    (effects (font (size 1.27 1.27)) (justify left))
-  )
-  (label "V_PMID" (at 295.91 170.18 0)
-    (effects (font (size 1.27 1.27)) (justify left))
-  )
-  (label "LSCTRL" (at 326.39 168.91 0)
-    (effects (font (size 1.27 1.27)) (justify left))
-  )
-  (label "SW" (at 295.91 167.64 0)
-    (effects (font (size 1.27 1.27)) (justify left))
-  )
-  (label "CC_#CD" (at 326.39 166.37 0)
-    (effects (font (size 1.27 1.27)) (justify left))
-  )
-  (label "GND" (at 295.91 165.1 0)
-    (effects (font (size 1.27 1.27)) (justify left))
-  )
-  (label "MR#" (at 326.39 163.83 0)
-    (effects (font (size 1.27 1.27)) (justify left))
-  )
-  (label "VCC" (at 295.91 162.56 0)
-    (effects (font (size 1.27 1.27)) (justify left))
-  )
-  (label "GND" (at 326.39 161.29 0)
-    (effects (font (size 1.27 1.27)) (justify left))
-  )
-  (label "VCC" (at 295.91 160.02 0)
-    (effects (font (size 1.27 1.27)) (justify left))
-  )
-  (label "CC_#PG" (at 326.39 158.75 0)
-    (effects (font (size 1.27 1.27)) (justify left))
-  )
-  (label "V_PMID" (at 295.91 157.48 0)
-    (effects (font (size 1.27 1.27)) (justify left))
-  )
-  (label "RESETN" (at 326.39 156.21 0)
-    (effects (font (size 1.27 1.27)) (justify left))
-  )
-  (label "V_PMID" (at 295.91 154.94 0)
-    (effects (font (size 1.27 1.27)) (justify left))
-  )
-  (label "INT" (at 326.39 153.67 0)
-    (effects (font (size 1.27 1.27)) (justify left))
-  )
-  (label "+1.8V" (at 295.91 152.4 0)
-    (effects (font (size 1.27 1.27)) (justify left))
-  )
-  (label "GND" (at 326.39 151.13 0)
-    (effects (font (size 1.27 1.27)) (justify left))
-  )
-  (label "GND" (at 295.91 149.86 0)
-    (effects (font (size 1.27 1.27)) (justify left))
-  )
-  (label "3V3" (at 326.39 148.59 0)
-    (effects (font (size 1.27 1.27)) (justify left))
-  )
-  (label "GND" (at 295.91 147.32 0)
-    (effects (font (size 1.27 1.27)) (justify left))
-  )
-  (label "$1N65" (at 326.39 146.05 0)
-    (effects (font (size 1.27 1.27)) (justify left))
-  )
-  (label "TS" (at 295.91 144.78 0)
     (effects (font (size 1.27 1.27)) (justify left))
   )
@@
     (effects (font (size 1.27 1.27)) (justify left))
   )
+  (label "TS" (at 289.84 263.81 0)
+    (effects (font (size 1.27 1.27)) (justify left))
+  )
+  (label "TP4056_PROG" (at 289.84 261.27 0)
+    (effects (font (size 1.27 1.27)) (justify left))
+  )
+  (label "GND" (at 289.84 258.73 0)
+    (effects (font (size 1.27 1.27)) (justify left))
+  )
+  (label "VUSB" (at 289.84 256.19 0)
+    (effects (font (size 1.27 1.27)) (justify left))
+  )
+  (label "VUSB" (at 310.16 263.81 0)
+    (effects (font (size 1.27 1.27)) (justify left))
+  )
+  (label "CC_#CD" (at 310.16 261.27 0)
+    (effects (font (size 1.27 1.27)) (justify left))
+  )
+  (label "CC_#PG" (at 310.16 258.73 0)
+    (effects (font (size 1.27 1.27)) (justify left))
+  )
+  (label "VCC" (at 310.16 256.19 0)
+    (effects (font (size 1.27 1.27)) (justify left))
+  )
+  (label "VCC" (at 289.84 303.81 0)
+    (effects (font (size 1.27 1.27)) (justify left))
+  )
+  (label "FB_1V8" (at 289.84 301.27 0)
+    (effects (font (size 1.27 1.27)) (justify left))
+  )
+  (label "GND" (at 289.84 298.73 0)
+    (effects (font (size 1.27 1.27)) (justify left))
+  )
+  (label "VCC" (at 310.16 301.27 0)
+    (effects (font (size 1.27 1.27)) (justify left))
+  )
+  (label "SW" (at 310.16 298.73 0)
+    (effects (font (size 1.27 1.27)) (justify left))
+  )
+  (label "GND" (at 310.16 296.19 0)
+    (effects (font (size 1.27 1.27)) (justify left))
+  )
+  (label "VCC" (at 289.84 337.54 0)
+    (effects (font (size 1.27 1.27)) (justify left))
+  )
+  (label "GND" (at 289.84 335 0)
+    (effects (font (size 1.27 1.27)) (justify left))
+  )
+  (label "LSCTRL" (at 289.84 332.46000000000004 0)
+    (effects (font (size 1.27 1.27)) (justify left))
+  )
+  (label "3V3" (at 310.16 337.54 0)
+    (effects (font (size 1.27 1.27)) (justify left))
+  )
+  (label "TP4056_PROG" (at 254.92 260 0)
+    (effects (font (size 1.27 1.27)) (justify left))
+  )
+  (label "GND" (at 265.08 260 0)
+    (effects (font (size 1.27 1.27)) (justify left))
+  )
+  (label "FB_1V8" (at 254.92 295 0)
+    (effects (font (size 1.27 1.27)) (justify left))
+  )
+  (label "+1.8V" (at 265.08 295 0)
+    (effects (font (size 1.27 1.27)) (justify left))
+  )
+  (label "FB_1V8" (at 254.92 305 0)
+    (effects (font (size 1.27 1.27)) (justify left))
+  )
+  (label "GND" (at 265.08 305 0)
+    (effects (font (size 1.27 1.27)) (justify left))
+  )
+  (label "CC_#CD" (at 334.92 250 0)
+    (effects (font (size 1.27 1.27)) (justify left))
+  )
+  (label "3V3" (at 345.08 250 0)
+    (effects (font (size 1.27 1.27)) (justify left))
+  )
+  (label "CC_#PG" (at 334.92 260 0)
+    (effects (font (size 1.27 1.27)) (justify left))
+  )
+  (label "3V3" (at 345.08 260 0)
+    (effects (font (size 1.27 1.27)) (justify left))
+  )
   (label "GND" (at 409.84 -0.9499999999999993 0)
     (effects (font (size 1.27 1.27)) (justify left))
@@
     )
   )
-  (symbol (lib_id "haven_dev_board:U2") (at 311.15 160.02 0) (unit 1)
-    (in_bom no) (on_board no)
-    (property "Reference" "U2" (at 311.15 155.02 0)
-      (effects (font (size 1.27 1.27)))
-    )
-    (property "Value" "BQ25120AYFPR" (at 311.15 165.02 0)
-      (effects (font (size 1.27 1.27)))
-    )
-  )
   (symbol (lib_id "haven_dev_board:U6") (at 341.63 69.85 0) (unit 1)
     (in_bom no) (on_board no)
@@
       (effects (font (size 1.27 1.27)))
     )
+  )
+  (symbol (lib_id "haven_dev_board:TP4056") (at 300 260 0) (unit 1)
+    (in_bom yes) (on_board yes)
+    (property "Reference" "U2" (at 300 248 0)
+      (effects (font (size 1.27 1.27)))
+    )
+    (property "Value" "TP4056" (at 300 272 0)
+      (effects (font (size 1.27 1.27)))
+    )
+  )
+  (symbol (lib_id "haven_dev_board:TPS62822DLC") (at 300 300 0) (unit 1)
+    (in_bom yes) (on_board yes)
+    (property "Reference" "U_BUCK1" (at 300 288 0)
+      (effects (font (size 1.27 1.27)))
+    )
+    (property "Value" "TPS62822DLCR" (at 300 312 0)
+      (effects (font (size 1.27 1.27)))
+    )
+  )
+  (symbol (lib_id "haven_dev_board:TPS22917") (at 300 335 0) (unit 1)
+    (in_bom yes) (on_board yes)
+    (property "Reference" "U_LS1" (at 300 323 0)
+      (effects (font (size 1.27 1.27)))
+    )
+    (property "Value" "TPS22917DBVR" (at 300 347 0)
+      (effects (font (size 1.27 1.27)))
+    )
+  )
+  (symbol (lib_id "haven_dev_board:R_PROG") (at 260 260 0) (unit 1)
+    (in_bom yes) (on_board yes)
+    (property "Reference" "R_PROG" (at 260 248 0)
+      (effects (font (size 1.27 1.27)))
+    )
+    (property "Value" "1.2k" (at 260 272 0)
+      (effects (font (size 1.27 1.27)))
+    )
+  )
+  (symbol (lib_id "haven_dev_board:R_FB1") (at 260 295 0) (unit 1)
+    (in_bom yes) (on_board yes)
+    (property "Reference" "R_FB1" (at 260 283 0)
+      (effects (font (size 1.27 1.27)))
+    )
+    (property "Value" "200k" (at 260 307 0)
+      (effects (font (size 1.27 1.27)))
+    )
+  )
+  (symbol (lib_id "haven_dev_board:R_FB2") (at 260 305 0) (unit 1)
+    (in_bom yes) (on_board yes)
+    (property "Reference" "R_FB2" (at 260 293 0)
+      (effects (font (size 1.27 1.27)))
+    )
+    (property "Value" "100k" (at 260 317 0)
+      (effects (font (size 1.27 1.27)))
+    )
+  )
+  (symbol (lib_id "haven_dev_board:R_PU_CHRG") (at 340 250 0) (unit 1)
+    (in_bom yes) (on_board yes)
+    (property "Reference" "R_PU_CHRG" (at 340 238 0)
+      (effects (font (size 1.27 1.27)))
+    )
+    (property "Value" "100k" (at 340 262 0)
+      (effects (font (size 1.27 1.27)))
+    )
+  )
+  (symbol (lib_id "haven_dev_board:R_PU_STDBY") (at 340 260 0) (unit 1)
+    (in_bom yes) (on_board yes)
+    (property "Reference" "R_PU_STDBY" (at 340 248 0)
+      (effects (font (size 1.27 1.27)))
+    )
+    (property "Value" "100k" (at 340 272 0)
+      (effects (font (size 1.27 1.27)))
+    )

Commit message: Actually remove U6 (BQ27220 fuel gauge) -- the TL;DR already claimed this
Found by cross-checking the full schematic+PCB reference list against
the doc's own claims: the TL;DR at the top of HARDWARE_COST_ALTERNATIVES.md
already says "fuel gauge dropped entirely -- confirmed nothing reads it,"
but that was a real decision (verified earlier by searching both app
repos for any fuel-gauge/battery-level reference and finding zero) that
had never actually been executed as a schematic/PCB edit. U6 was still
sitting on both files.

Removed the schematic instance + its 9 pin labels, and the PCB footprint.
Left two now-vestigial passives (R17, C23 -- bias/decoupling for U6's
BIN/VDD pins) in place rather than also removing them, same convention
as the earlier BQ25120A removal (which similarly left some now-unused
caps in place) -- correctly pruning a whole local bias network needs
more circuit understanding than "nothing reads this chip" covers.

kicad-cli sch erc: still 88 violations, unchanged (GND/VCC/SDA/SCL/V_BAT
are all shared with other components, no new dangling nets). kicad-cli
pcb drc: 222 vs. 215 -- the increase is exactly the expected "orphaned
trace stub" pattern (track_dangling +8, matching U6's pin count almost
exactly), not a new clearance or short (checked directly: clearance
count unchanged at 54, no shorting_items appeared).

Co-Authored-By: Claude Sonnet 5 <noreply@anthropic.com>
Claude-Session: https://claude.ai/code/session_01YTbrWH9Gt2quSDLgz6Te5V
Parts:
- removed U6: BQ27220YZFR, symbol haven_dev_board:U6
Changed lines of the file:
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@@
-    (effects (font (size 1.27 1.27)) (justify left))
-  )
-  (label "GPOUT" (at 326.39 80.01 0)
-    (effects (font (size 1.27 1.27)) (justify left))
-  )
-  (label "$1N74" (at 356.87 80.01 0)
-    (effects (font (size 1.27 1.27)) (justify left))
-  )
-  (label "SDA" (at 326.39 77.47 0)
-    (effects (font (size 1.27 1.27)) (justify left))
-  )
-  (label "GND" (at 356.87 77.47 0)
-    (effects (font (size 1.27 1.27)) (justify left))
-  )
-  (label "SCL" (at 326.39 74.93 0)
-    (effects (font (size 1.27 1.27)) (justify left))
-  )
-  (label "$1N70" (at 356.87 74.93 0)
-    (effects (font (size 1.27 1.27)) (justify left))
-  )
-  (label "V_BAT" (at 326.39 69.85 0)
-    (effects (font (size 1.27 1.27)) (justify left))
-  )
-  (label "VCC" (at 326.39 67.31 0)
-    (effects (font (size 1.27 1.27)) (justify left))
-  )
-  (label "V_BAT" (at 326.39 64.77 0)
     (effects (font (size 1.27 1.27)) (justify left))
   )
@@
     (effects (font (size 1.27 1.27)) (justify left))
   )
-  (label "MIC_IN" (at 369.84 -20.0 0)
-    (effects (font (size 1.27 1.27)) (justify left))
-  )
-  (label "GND" (at 390.16 -20.0 0)
+  (label "MIC_IN" (at 369.84 -20 0)
+    (effects (font (size 1.27 1.27)) (justify left))
+  )
+  (label "GND" (at 390.16 -20 0)
     (effects (font (size 1.27 1.27)) (justify left))
   )
@@
       (effects (font (size 1.27 1.27)))
     )
-  )
-  (symbol (lib_id "haven_dev_board:U6") (at 341.63 69.85 0) (unit 1)
-    (in_bom no) (on_board no)
-    (property "Reference" "U6" (at 341.63 64.85 0)
-      (effects (font (size 1.27 1.27)))
-    )
-    (property "Value" "BQ27220YZFR" (at 341.63 74.85 0)
-      (effects (font (size 1.27 1.27)))
-    )
