File: kicad/haven_dev_board.kicad_sch (KiCad schematic)
At the start: 90 parts, among them CN1 BM46B-12DS-0.35V(51), J1 CLE-107-01-G-DV, Q1 CSD23382F4, Q2 CSD13380F3T, Q3 CSD13380F3T, SW1 TS2819A 230GF, U1 BMI160, U10 SN74AXC4T774RSVR, U12 GT-USB-9047A, U13 SPH0641LU4H-1, U14 MX25R6435FBFIL0, U15 TAC5301QRGERQ1, U2 BQ25120AYFPR, U3 AP22916BCA4-7, U4 XL-0201SURC, U5 KTD2026, U6 BQ27220YZFR, U8 1MΩ, U9 AP22916BCA4-7, X1 Q13FC1350000200

Commit message: Fix a real bug: HVDD cannot be tied to 3V3, needs 5.6-12V
Caught this while researching the mic bias circuit (pulled the real
application note, SLAAED4, and the datasheet's own Recommended Operating
Conditions table). HVDD's actual spec is 5.6V MIN / 9V TYP / 12V MAX
(Section 5.3, "HVDD supply voltage to AVSS") -- tying it to the board's
3.3V rail, as stage 1 did, would put it below its functional minimum.
Given MICBIAS is generated internally from HVDD, this would very likely
have meant a mic bias output of ~0V on a built board, not "works but
suboptimal."

Fixed by disconnecting HVDD rather than leaving the wrong tie in place.
Identified a real, verified candidate for the actual fix (TPS61040-class
boost converter: SOT-23, single-Li-ion-cell input, sold specifically as a
"bias voltage" boost converter, output range covers HVDD's requirement,
and the current draw is tiny -- datasheet's own reference design shows
1.1mA at HVDD=11V) but the boost sub-circuit itself (inductor, diode,
feedback resistors) is not designed yet -- that's the next real task, not
done in this commit.

Also pulled the real mic bias circuit from SLAAED4 (TI's "Analog Input
Configurations" app note) and the datasheet's own Figure 8-1 reference
design (mono mic + mono lineout, matching Haven's exact topology): 2.2kΩ
bias resistor from MICBIAS to the mic (matches CMA-4544PF-W's own
datasheet test circuit exactly) and a 1µF AC-coupling cap into IN1P,
single-ended mode (IN1M unused). Component addition itself is the next
step, not yet in the schematic.

Co-Authored-By: Claude Sonnet 5 <noreply@anthropic.com>
Claude-Session: https://claude.ai/code/session_01YTbrWH9Gt2quSDLgz6Te5V
Changed lines of the file:
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@@
-    (effects (font (size 1.27 1.27)) (justify left))
-  )
-  (label "3V3" (at 447.04 110.49 0)
     (effects (font (size 1.27 1.27)) (justify left))
   )

Commit message: Stage 2: add the real mic bias network and decoupling caps
R29 (2.2kOhm, MICBIAS -> mic capsule): value matches CMA-4544PF-W's own
datasheet test circuit exactly, not a generic guess.
C50 (1uF, mic capsule -> codec IN1P): AC-coupling cap per TI app note
SLAAED4 Figure 2-1's reference circuit.
C51 (0.1uF, DREG -> GND) and C52 (1uF, VREF -> GND): both values from the
datasheet's own Figure 8-1 typical application circuit, not guessed.

Verified via real ERC (89 violations, up from stage 1's 88 -- identity-
diffed, not just counted). The one new entry is MIC_BIAS_NODE, exactly
the expected "fresh minimal net" reporting pattern already validated last
stage. DREG_DECOUPLE/VREF_DECOUPLE/MIC_BIAS remain individually flagged
even with their real second connections now in place -- traced this
through explicitly rather than waving it off: a decoupling cap's two legs
are two different nets by design (that's what makes it a decoupling cap),
so each net (DREG_DECOUPLE, VREF_DECOUPLE, MIC_BIAS) is still its own
small 2-member group, matching the same reporting pattern as before, not
a new problem.

Still not done: HVDD boost converter (see previous commit), MICBIAS's own
decoupling cap (low priority until HVDD exists), OUT2P/OUT2M termination,
all PCB footprint/routing work.

Co-Authored-By: Claude Sonnet 5 <noreply@anthropic.com>
Claude-Session: https://claude.ai/code/session_01YTbrWH9Gt2quSDLgz6Te5V
Parts:
- added C50: 1uF_couple, symbol haven_dev_board:C_1uF_couple
- added C51: 0.1uF_dreg, symbol haven_dev_board:C_0.1uF_dreg
- added C52: 1uF_vref, symbol haven_dev_board:C_1uF_vref
- added R29: 2.2k, symbol haven_dev_board:R_2.2k
Changed lines of the file:
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@@
     (effects (font (size 1.27 1.27)) (justify left))
   )
-  (label "MIC_P" (at 430.53 175.0 0)
-    (effects (font (size 1.27 1.27)) (justify left))
-  )
-  (label "GND" (at 443.23 175.0 0)
+  (label "MIC_BIAS_NODE" (at 430.53 175 0)
+    (effects (font (size 1.27 1.27)) (justify left))
+  )
+  (label "GND" (at 443.23 175 0)
+    (effects (font (size 1.27 1.27)) (justify left))
+  )
+  (label "MIC_BIAS" (at 460.0 145.08 0)
+    (effects (font (size 1.27 1.27)) (justify left))
+  )
+  (label "MIC_BIAS_NODE" (at 460.0 134.92 0)
+    (effects (font (size 1.27 1.27)) (justify left))
+  )
+  (label "MIC_BIAS_NODE" (at 470.0 145.08 0)
+    (effects (font (size 1.27 1.27)) (justify left))
+  )
+  (label "MIC_P" (at 470.0 134.92 0)
+    (effects (font (size 1.27 1.27)) (justify left))
+  )
+  (label "DREG_DECOUPLE" (at 480.0 145.08 0)
+    (effects (font (size 1.27 1.27)) (justify left))
+  )
+  (label "GND" (at 480.0 134.92 0)
+    (effects (font (size 1.27 1.27)) (justify left))
+  )
+  (label "VREF_DECOUPLE" (at 490.0 145.08 0)
+    (effects (font (size 1.27 1.27)) (justify left))
+  )
+  (label "GND" (at 490.0 134.92 0)
     (effects (font (size 1.27 1.27)) (justify left))
   )
@@
     )
   )
-  (symbol (lib_id "haven_dev_board:CMA-4544PF-W") (at 436.88 175.0 0) (unit 1)
-    (in_bom no) (on_board no)
-    (property "Reference" "MIC1" (at 436.88 170.0 0)
-      (effects (font (size 1.27 1.27)))
-    )
-    (property "Value" "CMA-4544PF-W" (at 436.88 180.0 0)
-      (effects (font (size 1.27 1.27)))
-    )
+  (symbol (lib_id "haven_dev_board:CMA-4544PF-W") (at 436.88 175 0) (unit 1)
+    (in_bom no) (on_board no)
+    (property "Reference" "MIC1" (at 436.88 170 0)
+      (effects (font (size 1.27 1.27)))
+    )
+    (property "Value" "CMA-4544PF-W" (at 436.88 180 0)
+      (effects (font (size 1.27 1.27)))
+    )
+  )
+  (symbol (lib_id "haven_dev_board:R_2.2k") (at 460.0 140.0 0) (unit 1)
+    (in_bom no) (on_board no)
+    (property "Reference" "R29" (at 457.46 145.08 0)
+      (effects (font (size 1.27 1.27)))
+    )
+    (property "Value" "2.2k" (at 457.46 134.92 0)
+      (effects (font (size 1.27 1.27)))
+    )
+  )
+  (symbol (lib_id "haven_dev_board:C_1uF_couple") (at 470.0 140.0 0) (unit 1)
+    (in_bom no) (on_board no)
+    (property "Reference" "C50" (at 467.46 145.08 0)
+      (effects (font (size 1.27 1.27)))
+    )
+    (property "Value" "1uF_couple" (at 467.46 134.92 0)
+      (effects (font (size 1.27 1.27)))
+    )
+  )
+  (symbol (lib_id "haven_dev_board:C_0.1uF_dreg") (at 480.0 140.0 0) (unit 1)
+    (in_bom no) (on_board no)
+    (property "Reference" "C51" (at 477.46 145.08 0)
+      (effects (font (size 1.27 1.27)))
+    )
+    (property "Value" "0.1uF_dreg" (at 477.46 134.92 0)
+      (effects (font (size 1.27 1.27)))
+    )
+  )
+  (symbol (lib_id "haven_dev_board:C_1uF_vref") (at 490.0 140.0 0) (unit 1)
+    (in_bom no) (on_board no)
+    (property "Reference" "C52" (at 487.46 145.08 0)
+      (effects (font (size 1.27 1.27)))
+    )
+    (property "Value" "1uF_vref" (at 487.46 134.92 0)
+      (effects (font (size 1.27 1.27)))
+    )

Commit message: Stage 3: HVDD boost converter (TPS61040), real reference design
Solves the HVDD-needs-5.6-12V bug from the previous commit. Real
reference design: TI TPS61040 datasheet (SLVS413L) Figure 7-1, an
18V-from-battery boost converter using exactly this topology -- kept
every component value except the feedback divider, which is recomputed
for Haven's 9V target (mid-range of the required 5.6-12V) using the
datasheet's own formula: VOUT = 1.233V * (1 + R1/R2). R2 kept at the
reference design's 160kOhm; solved R1 = 1.0Mohm, giving ~8.94V -- checked
against the requirement, not assumed.

L1 (10uH), D1 (MBR0530), CFF (22pF), C1 (4.7uF in), C2 (1uF out): all the
reference design's own values, unmodified. Haven's actual HVDD load
(~1.1mA per the TAC5301-Q1 datasheet's own reference design) is far below
the reference design's 10mA target, so these are safe with margin, not
re-optimized for headroom I don't need.

ERC identity-diffed against stage 2: exactly 3 new entries (HVDD, SW_NODE,
FB_NODE), each the expected single-representative report for a freshly
introduced, multi-member net -- same pattern validated twice already, not
a new anomaly.

EN tied directly to V_BAT (always-on) -- a real scope simplification,
noted in the script docstring, not hidden.

Real remaining open items: inductor/diode real stock check, PCB layout
(switching converter SW-node copper is layout-sensitive, schematic-correct
isn't layout-correct), OUT2P/OUT2M termination, MICBIAS's own decoupling
cap, and all PCB footprint placement/routing.

Co-Authored-By: Claude Sonnet 5 <noreply@anthropic.com>
Claude-Session: https://claude.ai/code/session_01YTbrWH9Gt2quSDLgz6Te5V
Parts:
- added C53: 4.7uF_in, symbol haven_dev_board:C_4.7uF_in
- added C54: 1uF_out, symbol haven_dev_board:C_1uF_out
- added C55: 22pF_ff, symbol haven_dev_board:C_22pF_ff
- added D1: MBR0530, symbol haven_dev_board:D_MBR0530
- added L1: 10uH, symbol haven_dev_board:L_10uH
- added R30: 1.0M, symbol haven_dev_board:R_1.0M
- added R31: 160k, symbol haven_dev_board:R_160k
- added U16: TPS61040DBVR, symbol haven_dev_board:TPS61040
Changed lines of the file:
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@@
     (effects (font (size 1.27 1.27)) (justify left))
   )
-  (label "MIC_BIAS" (at 460.0 145.08 0)
-    (effects (font (size 1.27 1.27)) (justify left))
-  )
-  (label "MIC_BIAS_NODE" (at 460.0 134.92 0)
-    (effects (font (size 1.27 1.27)) (justify left))
-  )
-  (label "MIC_BIAS_NODE" (at 470.0 145.08 0)
-    (effects (font (size 1.27 1.27)) (justify left))
-  )
-  (label "MIC_P" (at 470.0 134.92 0)
-    (effects (font (size 1.27 1.27)) (justify left))
-  )
-  (label "DREG_DECOUPLE" (at 480.0 145.08 0)
-    (effects (font (size 1.27 1.27)) (justify left))
-  )
-  (label "GND" (at 480.0 134.92 0)
-    (effects (font (size 1.27 1.27)) (justify left))
-  )
-  (label "VREF_DECOUPLE" (at 490.0 145.08 0)
-    (effects (font (size 1.27 1.27)) (justify left))
-  )
-  (label "GND" (at 490.0 134.92 0)
+  (label "MIC_BIAS" (at 460 145.08 0)
+    (effects (font (size 1.27 1.27)) (justify left))
+  )
+  (label "MIC_BIAS_NODE" (at 460 134.92 0)
+    (effects (font (size 1.27 1.27)) (justify left))
+  )
+  (label "MIC_BIAS_NODE" (at 470 145.08 0)
+    (effects (font (size 1.27 1.27)) (justify left))
+  )
+  (label "MIC_P" (at 470 134.92 0)
+    (effects (font (size 1.27 1.27)) (justify left))
+  )
+  (label "DREG_DECOUPLE" (at 480 145.08 0)
+    (effects (font (size 1.27 1.27)) (justify left))
+  )
+  (label "GND" (at 480 134.92 0)
+    (effects (font (size 1.27 1.27)) (justify left))
+  )
+  (label "VREF_DECOUPLE" (at 490 145.08 0)
+    (effects (font (size 1.27 1.27)) (justify left))
+  )
+  (label "GND" (at 490 134.92 0)
+    (effects (font (size 1.27 1.27)) (justify left))
+  )
+  (label "SW_NODE" (at 539.84 145.08 0)
+    (effects (font (size 1.27 1.27)) (justify left))
+  )
+  (label "GND" (at 539.84 134.92 0)
+    (effects (font (size 1.27 1.27)) (justify left))
+  )
+  (label "FB_NODE" (at 560.16 134.92 0)
+    (effects (font (size 1.27 1.27)) (justify left))
+  )
+  (label "V_BAT" (at 560.16 140.0 0)
+    (effects (font (size 1.27 1.27)) (justify left))
+  )
+  (label "V_BAT" (at 560.16 145.08 0)
+    (effects (font (size 1.27 1.27)) (justify left))
+  )
+  (label "V_BAT" (at 520.0 115.08 0)
+    (effects (font (size 1.27 1.27)) (justify left))
+  )
+  (label "SW_NODE" (at 520.0 104.92 0)
+    (effects (font (size 1.27 1.27)) (justify left))
+  )
+  (label "SW_NODE" (at 560.0 115.08 0)
+    (effects (font (size 1.27 1.27)) (justify left))
+  )
+  (label "HVDD" (at 560.0 104.92 0)
+    (effects (font (size 1.27 1.27)) (justify left))
+  )
+  (label "V_BAT" (at 535.0 165.08 0)
+    (effects (font (size 1.27 1.27)) (justify left))
+  )
+  (label "GND" (at 535.0 154.92 0)
+    (effects (font (size 1.27 1.27)) (justify left))
+  )
+  (label "HVDD" (at 580.0 145.08 0)
+    (effects (font (size 1.27 1.27)) (justify left))
+  )
+  (label "GND" (at 580.0 134.92 0)
+    (effects (font (size 1.27 1.27)) (justify left))
+  )
+  (label "HVDD" (at 580.0 175.08 0)
+    (effects (font (size 1.27 1.27)) (justify left))
+  )
+  (label "FB_NODE" (at 580.0 164.92 0)
+    (effects (font (size 1.27 1.27)) (justify left))
+  )
+  (label "FB_NODE" (at 580.0 205.08 0)
+    (effects (font (size 1.27 1.27)) (justify left))
+  )
+  (label "GND" (at 580.0 194.92 0)
+    (effects (font (size 1.27 1.27)) (justify left))
+  )
+  (label "HVDD" (at 595.0 175.08 0)
+    (effects (font (size 1.27 1.27)) (justify left))
+  )
+  (label "FB_NODE" (at 595.0 164.92 0)
     (effects (font (size 1.27 1.27)) (justify left))
   )
@@
     )
   )
-  (symbol (lib_id "haven_dev_board:R_2.2k") (at 460.0 140.0 0) (unit 1)
+  (symbol (lib_id "haven_dev_board:R_2.2k") (at 460 140 0) (unit 1)
     (in_bom no) (on_board no)
     (property "Reference" "R29" (at 457.46 145.08 0)
@@
     )
   )
-  (symbol (lib_id "haven_dev_board:C_1uF_couple") (at 470.0 140.0 0) (unit 1)
+  (symbol (lib_id "haven_dev_board:C_1uF_couple") (at 470 140 0) (unit 1)
     (in_bom no) (on_board no)
     (property "Reference" "C50" (at 467.46 145.08 0)
@@
     )
   )
-  (symbol (lib_id "haven_dev_board:C_0.1uF_dreg") (at 480.0 140.0 0) (unit 1)
+  (symbol (lib_id "haven_dev_board:C_0.1uF_dreg") (at 480 140 0) (unit 1)
     (in_bom no) (on_board no)
     (property "Reference" "C51" (at 477.46 145.08 0)
@@
     )
   )
-  (symbol (lib_id "haven_dev_board:C_1uF_vref") (at 490.0 140.0 0) (unit 1)
+  (symbol (lib_id "haven_dev_board:C_1uF_vref") (at 490 140 0) (unit 1)
     (in_bom no) (on_board no)
     (property "Reference" "C52" (at 487.46 145.08 0)
@@
       (effects (font (size 1.27 1.27)))
     )
+  )
+  (symbol (lib_id "haven_dev_board:TPS61040") (at 550.0 140.0 0) (unit 1)
+    (in_bom no) (on_board no)
+    (property "Reference" "U16" (at 550.0 128.0 0)
+      (effects (font (size 1.27 1.27)))
+    )
+    (property "Value" "TPS61040DBVR" (at 550.0 152.0 0)
+      (effects (font (size 1.27 1.27)))
+    )
+  )
+  (symbol (lib_id "haven_dev_board:L_10uH") (at 520.0 110.0 0) (unit 1)
+    (in_bom no) (on_board no)
+    (property "Reference" "L1" (at 517.46 115.08 0)
+      (effects (font (size 1.27 1.27)))
+    )
+    (property "Value" "10uH" (at 517.46 104.92 0)
+      (effects (font (size 1.27 1.27)))
+    )
+  )
+  (symbol (lib_id "haven_dev_board:D_MBR0530") (at 560.0 110.0 0) (unit 1)
+    (in_bom no) (on_board no)
+    (property "Reference" "D1" (at 557.46 115.08 0)
+      (effects (font (size 1.27 1.27)))
+    )
+    (property "Value" "MBR0530" (at 557.46 104.92 0)
+      (effects (font (size 1.27 1.27)))
+    )
+  )
+  (symbol (lib_id "haven_dev_board:C_4.7uF_in") (at 535.0 160.0 0) (unit 1)
+    (in_bom no) (on_board no)
+    (property "Reference" "C53" (at 532.46 165.08 0)
+      (effects (font (size 1.27 1.27)))
+    )
+    (property "Value" "4.7uF_in" (at 532.46 154.92 0)
+      (effects (font (size 1.27 1.27)))
+    )
+  )
+  (symbol (lib_id "haven_dev_board:C_1uF_out") (at 580.0 140.0 0) (unit 1)
+    (in_bom no) (on_board no)
+    (property "Reference" "C54" (at 577.46 145.08 0)
+      (effects (font (size 1.27 1.27)))
+    )
+    (property "Value" "1uF_out" (at 577.46 134.92 0)
+      (effects (font (size 1.27 1.27)))
+    )
+  )
+  (symbol (lib_id "haven_dev_board:R_1.0M") (at 580.0 170.0 0) (unit 1)
+    (in_bom no) (on_board no)
+    (property "Reference" "R30" (at 577.46 175.08 0)
+      (effects (font (size 1.27 1.27)))
+    )
+    (property "Value" "1.0M" (at 577.46 164.92 0)
+      (effects (font (size 1.27 1.27)))
+    )
+  )
+  (symbol (lib_id "haven_dev_board:R_160k") (at 580.0 200.0 0) (unit 1)
+    (in_bom no) (on_board no)
+    (property "Reference" "R31" (at 577.46 205.08 0)
+      (effects (font (size 1.27 1.27)))
+    )
+    (property "Value" "160k" (at 577.46 194.92 0)
+      (effects (font (size 1.27 1.27)))
+    )
+  )
+  (symbol (lib_id "haven_dev_board:C_22pF_ff") (at 595.0 170.0 0) (unit 1)
+    (in_bom no) (on_board no)
+    (property "Reference" "C55" (at 592.46 175.08 0)
+      (effects (font (size 1.27 1.27)))
+    )
+    (property "Value" "22pF_ff" (at 592.46 164.92 0)
+      (effects (font (size 1.27 1.27)))
+    )

Commit message: Add MICBIAS decoupling cap, fold into the stage-3 script for reproducibility
C56 (1uF, 35V rated): value straight from the TAC5301-Q1 datasheet's own
Figure 8-1 reference circuit. Regenerated all three stages from a clean
baseline to confirm the consolidated script reproduces the identical
result (92 violations, matching the manual add this replaces).

This closes out the schematic-level open items from the last two commits
(OUT2P/OUT2M: left genuinely unconnected, which is standard practice for
an unused differential audio output, and this project's ERC ruleset has
no "unused pin" check to satisfy either way -- confirmed by checking, not
assumed). Schematic is now complete for what stage 1-3 set out to do.

Co-Authored-By: Claude Sonnet 5 <noreply@anthropic.com>
Claude-Session: https://claude.ai/code/session_01YTbrWH9Gt2quSDLgz6Te5V
Parts:
- added C56: 1uF_35V_micbias, symbol haven_dev_board:C_1uF_35V_micbias
Changed lines of the file:
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@@
     (effects (font (size 1.27 1.27)) (justify left))
   )
+  (label "MIC_BIAS" (at 610.0 145.08 0)
+    (effects (font (size 1.27 1.27)) (justify left))
+  )
+  (label "GND" (at 610.0 134.92 0)
+    (effects (font (size 1.27 1.27)) (justify left))
+  )
   (symbol (lib_id "haven_dev_board:U1") (at 210.82 193.04 0) (unit 1)
     (in_bom no) (on_board no)
@@
       (effects (font (size 1.27 1.27)))
     )
+  )
+  (symbol (lib_id "haven_dev_board:C_1uF_35V_micbias") (at 610.0 140.0 0) (unit 1)
+    (in_bom no) (on_board no)
+    (property "Reference" "C56" (at 607.46 145.08 0)
+      (effects (font (size 1.27 1.27)))
+    )
+    (property "Value" "1uF_35V_micbias" (at 607.46 134.92 0)
+      (effects (font (size 1.27 1.27)))
+    )
