File: kicad/haven_dev_board.kicad_sch (KiCad schematic)
At the start: 89 parts, among them CN1 BM46B-12DS-0.35V(51), J1 CLE-107-01-G-DV, Q1 CSD23382F4, Q2 CSD13380F3T, Q3 CSD13380F3T, SW1 TS2819A 230GF, U1 BMI160, U10 SN74AXC4T774RSVR, U12 GT-USB-9047A, U13 SPH0641LU4H-1, U14 MX25R6435FBFIL0, U15 ADAU1860BCBZRL, U2 BQ25120AYFPR, U3 AP22916BCA4-7, U4 XL-0201SURC, U5 KTD2026, U6 BQ27220YZFR, U8 1MΩ, U9 AP22916BCA4-7, X1 Q13FC1350000200

Commit message: Make the port's schematic load in KiCad so BOM export works
kicad-cli returned zero BOM rows and an empty netlist because KiCad loaded
no symbols at all: the embedded lib_symbols were named "U1" while placed
symbols referenced "haven_dev_board:U1". Placed symbols also lacked
in_bom/on_board, a Footprint property and an (instances ...) block.
tools/repair_schematic.py fixes all of these (footprints taken from the
board). BOM export now lists all 89 parts.

ERC goes from 84 to 208, which is ERC finally seeing the symbols: 152
pin_not_connected + 55 label_dangling, because the generator placed net
labels near pins rather than on them. Board nets come from OpenEarable's
own per-pad data, so this doesn't affect fabrication; it does mean the
schematic is documentation, not a source of connectivity, until labels
are snapped to pins.

Co-Authored-By: Claude Opus 5.5 <noreply@anthropic.com>
Claude-Session: https://claude.ai/code/session_01YTbrWH9Gt2quSDLgz6Te5V
Parts:
- C1, C10, C11, C12, C13, C14, C17, C19, C2, C21, C22, C23, C26, C27, C28, C29, C3, C31, C32, C36, C38, C4, C40, C42, C43, C44, C47, C48, C5, C6, C7, C9: footprint (none) -> haven_footprints:C0201
- C16, C18, C20, C33, C34, C41, C8: footprint (none) -> haven_footprints:C0402
- C45, C46: footprint (none) -> haven_footprints:b5c2858cad4e462ab76a8d0ccf4ade45
- C49: footprint (none) -> haven_footprints:cef4f92115b54348803d28f8706b0456
- CARD1: footprint (none) -> haven_footprints:TF-SMD_TF-06A
- CN1: footprint (none) -> haven_footprints:FPC-SMD_12P-P0.35_BM46B-12DS-0.35V
- CRYSTAL1: footprint (none) -> haven_footprints:6684822644394e4eba542a27714dd8a6
- D2: footprint (none) -> haven_footprints:SON-6_L1.5-W1.0-P0.50-BL
- J1: footprint (none) -> haven_footprints:CLE-107-01-X-DV
- L2: footprint (none) -> haven_footprints:L0402
- LED3: footprint (none) -> haven_footprints:LED-ARRAY-SMD_4P-L1.0-W1.0-TR-RD
- MDBT531: footprint (none) -> haven_footprints:MDBT53
- Q1: footprint (none) -> haven_footprints:PICOSTAR-3_L1.0-W0.6-P0.35-TL
- Q2, Q3: footprint (none) -> haven_footprints:PICOSTAR-3_L0.7-W0.6-P0.40-TL
- R1, R10, R11, R15, R17, R19, R2, R20, R23, R26, R27, R3, R4, R5, R6, R7, R8, R9, U8: footprint (none) -> haven_footprints:R0201
- R13, R21: footprint (none) -> haven_footprints:R0402
- R28: footprint (none) -> haven_footprints:ea94e26560f84db4a6862024f5c3efa7
- SW1: footprint (none) -> haven_footprints:SW-SMD_4P-L2.8-W1.9-P1.16-LS3.0
- U1: footprint (none) -> haven_footprints:LGA-14_L3.0-W2.5-P0.50-BL
- U10: footprint (none) -> haven_footprints:UQFN-16_L2.6-W1.8-P0.40-BL
- U12: footprint (none) -> haven_footprints:USB-C-SMD_GT-USB-9047A
- U13: footprint (none) -> haven_footprints:MIC-SMD_5P_L3.5-W2.7-P0.82_SPH0641LU4H-1
- U14: footprint (none) -> haven_footprints:WLCSP-22_MX25R6435FBFIL0
- U15: footprint (none) -> haven_footprints:BGA-56_L3.0-W2.7-P0.35-R8-C7-TL
- U2: footprint (none) -> haven_footprints:DSBGA-25_L2.5-W2.6-R5-C5-P0.40-BL
- U3, U9: footprint (none) -> haven_footprints:X1-WLB0808-4_L0.8-W0.8-P0.40-TL
- U4: footprint (none) -> haven_footprints:LED-SMD_L0.65-W0.35-P0.41_XL-0201SURC
- U5: footprint (none) -> haven_footprints:DFN-8_L1.5-W1.5-P0.40-BL-EP
- U6: footprint (none) -> haven_footprints:DSBGA-9_L1.7-W1.6-R3-C3-P0.50-BL
- X1: footprint (none) -> haven_footprints:FC-135R_L3.2-W1.5
Connections:
- net #ERROR: now also Q2.1 (G), U8.1
- net $1N117: now also Q2.2 (S), R4.1
- net $1N119: now also R4.2, U4.2 (K)
- net $1N151: now also C31.1, C36.1
- net $1N16368: now also C45.2, CRYSTAL1.2 (GND), R28.1
- net $1N2586: now also C32.1, U15.B8 (QSPIM_CLK/MP11)
- net $1N36: now also CARD1.2 (CS), R19.2
- net $1N48: now also R7.2, U12.B6 (DP2)
- net $1N49: now also R8.2, U12.A4B9 (VBUS)
- net $1N65: now also C10.2, U2.E5 (SCL)
- net $1N70: now also C23.1
- net $1N74: now also R17.1
- net $1N98: now also C3.2, R27.2
- net +1.8V: now also C1.1, C18.2, C20.1, C4.2, J1.5, L2.2, R2.1, R3.1, U2.A4 (SW)
- net 3V3: now also C17.2, C29.1, C48.2, C5.1, CN1.21, J1.6, U2.E4 (SDA), U4.1 (A), U5.9 (EP)
- net BCLK: now also U15.D2 (UART_COMM_TX/MP17)
- net CC_#CD: now also U2.D2 (INT)
- net CC_#PG: now also U2.D5 (GND)
- net DAC_N: now also U15.A6 (TMS/MP23)
- net DAC_P: now also U15.A5 (TCK/MP22)
- net DIN: now also U15.G5 (AINN2)
- net DOUT: now also U15.G8 (AINN0)
- net FLASH_RESET: now also U14.A2 (NC)
- net GND: now also C1.2, C10.1, C11.1, C12.2, C13.1, C14.2, C16.1, C17.1, C18.1, C19.1, C2.2, C20.2, C21.2, C22.1, C23.2, C26.1, C27.2, C28.1, C29.2, C3.1, C31.2, C32.2, C33.1, C34.2, C36.2, C38.2, C4.1, C40.2, C41.2, C42.1, C43.2, C44.2, C45.1, C46.2, C47.2, C48.1, C49.2, C5.2, C6.1, C7.1, C8.2, C9.1, CARD1.10 (EH), CARD1.11 (EH), CARD1.12 (EH), CARD1.13 (EH), CARD1.4 (VDD), CRYSTAL1.1, CRYSTAL1.3, D2.2 (GND), J1.7, Q2.3 (D), Q3.3 (D), R1.2, R17.2, R19.1, R6.1, R7.1, R8.1, SW1.1 (A), SW1.2 (A&apos;), U1.1 (SDO), U1.2 (ASDX), U1.5 (VDDIO), U1.6 (GNDIO), U1.7 (GND), U10.1 (A1), U10.3 (A3), U12.A9B4 (VBUS), U13.1 (DATA), U13.2 (SELECT), U14.A4 (NC), U15.B6 (XTALO), U15.B7 (XTALI/MCLKIN), U15.C7 (SCL/SCLK), U15.F3 (REG_EN), U2.A2 (IN), U2.A3 (PMID), U2.B4 (VINLS), U2.C3 (TS), U2.D4 (PG#), U2.E3 (LSCTRL), U3.B1 (GND), U5.5 (VIN), U5.6 (SCL), U8.2, U9.B1 (GND)
- net INT: now also U2.E2 (CD#)
- net IO1: now also J1.3
- net IO2: now also J1.4
- net IO3: now also J1.2
- net IO4: now also CN1.20
- net IO5: now also CN1.22
- net IO6: now also CN1.24
- net LRCLK: now also U15.A7 (TDO/MP24)
- net LSCTRL: now also U2.D1 (IPRETERM)
- net MR#: now also Q1.1 (G), SW1.3 (B), SW1.4 (B&apos;), U2.D3 (RESET)
- net PDMCLK: now also CN1.19, U13.5 (VDD), U15.D8 (QSPIM_SDIO1/MP14)
- net PDMDIN: now also CN1.17, U13.3 (GROUND), U15.E7 (QSPIM_SDIO3/MP16)
- net RESETN: now also C49.1, J1.9, U2.E1 (MR#)
- net RGB_B: now also U5.2 (D3)
- net RGB_G: now also U5.1 (ST)
- net SCL: now also R3.2, U2.C4 (VINLS), U5.8 (GND), U6.C3 (BAT)
- net SCL1: now also CN1.16, R9.2, U15.A1 (ROM_BOOT_MODE/MP21)
- net SCL2: now also R10.2, U1.9 (INT2)
- net SDA: now also R2.2, U2.C5 (LS/LDO), U5.7 (SDA)
- net SDA1: now also CN1.15, R5.2, U15.F6 (AINP0)
- net SDA2: now also CN1.23, R11.2, U1.8 (VDD)
- net SD_ENABLE: now also U9.B2 (ON)
- net SD_STATE: now also Q3.2 (S)
- net SD_STATE_3V3: now also CARD1.1 (RSV), Q3.1 (G), R1.1
- net SENSORS_ENABLE: now also U3.B2 (ON)
- net SPI_CLK: now also U10.6 (DIR4), U14.K5 (NC)
- net SPI_CLK_SD: now also CARD1.5 (SCLK), U10.15 (DIR1)
- net SPI_CS: now also U10.2 (A2), U10.8 (GND)
- net SPI_CS_FLASH: now also U14.B1 (NC)
- net SPI_CS_SD: now also CARD1.8 (RSV), R20.1, U10.13 (VCCB)
- net SPI_MISO: now also U10.5 (DIR3), U14.L4 (NC)
- net SPI_MISO_SD: now also CARD1.3 (DI), R15.2, U10.16 (DIR2)
- net SPI_MOSI: now also U10.7 (OE#), U14.L2 (NC)
- net SPI_MOSI_SD: now also CARD1.7 (DO), U10.14 (VCCA)
- net SW: now also L2.1, U2.B5 (SYS)
- net SWCLK: now also J1.13
- net SWDIO: now also J1.11
- net TCK: now also J1.8, U15.F2 (HPOUTP)
- net TDI: now also J1.14, U15.E5 (FSYNC_1/MP8)
- net TDO: now also J1.12, U15.C2 (FSYNC_0/MP4)
- net TMS: now also J1.10, U15.G1 (HPOUTN)
- net TS: now also R13.1, R6.2, U2.A1 (GND)
- net USB_D+: now also R23.2
- net USB_D-: now also R26.2
- net USB_DM: now also D2.3 (IO2), D2.4 (IO2), R26.1, U12.A7 (DN1), U12.B7 (DN2)
- net USB_DP: now also D2.1 (IO1), D2.6 (IO1), R23.1, U12.A5 (CC1), U12.A6 (DP1)
- net VCC: now also C19.2, R21.2, U2.B2 (BAT), U2.B3 (PMID)
- net VUSB: now also C22.2, D2.5 (VCC), R13.2, R27.1, U12.A1B12 (GND), U12.B5 (CC2), U2.C2 (ILIM)
- net V_BAT: now also C21.1, R21.1, U6.A3 (SCL), U6.C1 (SRP)
- net V_LS: now also C11.2, C12.1, C13.2, C27.1, C33.2, C34.1, C38.1, C40.1, C41.1, C42.2, C43.1, C44.1, C47.1, C7.2, CN1.18, J1.1, R10.1, R11.1, R5.1, R9.1, U1.10 (OCSB), U1.14 (SDX), U1.3 (ASCX), U10.10 (B3), U10.11 (B2), U10.4 (A4), U10.9 (B4), U13.4 (CLOCK), U14.B3 (NC), U14.K3 (NC), U15.E6 (SELFBOOT/MP19)
- net V_PMID: now also C16.2, C9.2, U2.A5 (PGND), U2.B1 (BAT), U2.C1 (ISET)
- net V_SD: now also C26.2, C28.2, C6.2, C8.1, CARD1.6 (VSS), R15.1, R20.2, U10.12 (B1)
- net XL1: now also C14.1, X1.1
- net XL2: now also C2.1, X1.2
- net XTALI: now also C46.1, CRYSTAL1.4 (GND), U15.D7 (ADDR1/MOSI/UART_CTRL_RX)
- net XTALO: now also R28.2, U15.D6 (ADDR0/SS#)

Commit message: Rev A: remove the OpenEarable parts Haven doesn't use
Deletes the microSD path (CARD1, U10 level shifter, U9 load switch, Q3/R1
card detect, R15/R20 pull-ups, V_SD decoupling C6/C8/C26/C28), the flash
(U14), the IMU (U1 and its SCL2/SDA2 pull-ups R10/R11), the fuel gauge (U6
with R17/C23/R19) and the flex-board connector CN1 (Hirose, 112-week lead
time). R21, the fuel gauge's 10 mOhm sense resistor in the battery path,
becomes a 0R jumper on the same footprint. J1 (Samtec SWD/JTAG) is
do-not-populate: its pads stay routed to SWDIO/SWCLK/RESETN/+1.8V/GND and
serve as programming test pads, avoiding new routing for a Tag-Connect.

U3 stays: it switches V_LS, which powers the ADAU1860 and the mic, so
firmware must drive SENSORS_ENABLE high.

Copper: 23 nets with no remaining pair of pads lose all tracks/vias;
affected nets that stay alive lose only stubs that KiCad's connectivity
engine reports dangling. 347 segments and 54 vias removed.

Outline unchanged (14.73 x 32.33 mm): the remaining copper at the old CN1
end (C48, codec I2C SDA1/SCL1, mic PDM) reaches 76.47 mm against a 77.41 mm
edge, so trimming gains under 0.6 mm and would break the enclosure fit.

DRC (zones filled): 0 unconnected, 0 shorts, 0 dangling tracks. BOM: 68
parts.

Co-Authored-By: Claude Opus 5.5 <noreply@anthropic.com>
Claude-Session: https://claude.ai/code/session_01YTbrWH9Gt2quSDLgz6Te5V
Parts:
- removed C23: 2.2uF, haven_footprints:C0201, symbol haven_dev_board:C23
- removed C26: 100nF, haven_footprints:C0201, symbol haven_dev_board:C26
- removed C28: 1uF, haven_footprints:C0201, symbol haven_dev_board:C28
- removed C6: 100nF, haven_footprints:C0201, symbol haven_dev_board:C6
- removed C8: 10uF, haven_footprints:C0402, symbol haven_dev_board:C8
- removed CARD1: TF-06A, haven_footprints:TF-SMD_TF-06A, symbol haven_dev_board:CARD1
- removed CN1: BM46B-12DS-0.35V(51), haven_footprints:FPC-SMD_12P-P0.35_BM46B-12DS-0.35V, symbol haven_dev_board:CN1
- removed Q3: CSD13380F3T, haven_footprints:PICOSTAR-3_L0.7-W0.6-P0.40-TL, symbol haven_dev_board:Q3
- removed R1: 10kΩ, haven_footprints:R0201, symbol haven_dev_board:R1
- removed R10: 2kΩ, haven_footprints:R0201, symbol haven_dev_board:R10
- removed R11: 2kΩ, haven_footprints:R0201, symbol haven_dev_board:R11
- removed R15: 10kΩ, haven_footprints:R0201, symbol haven_dev_board:R15
- removed R17: 10kΩ, haven_footprints:R0201, symbol haven_dev_board:R17
- removed R19: 10kΩ, haven_footprints:R0201, symbol haven_dev_board:R19
- removed R20: 10kΩ, haven_footprints:R0201, symbol haven_dev_board:R20
- removed U1: BMI160, haven_footprints:LGA-14_L3.0-W2.5-P0.50-BL, symbol haven_dev_board:U1
- removed U10: SN74AXC4T774RSVR, haven_footprints:UQFN-16_L2.6-W1.8-P0.40-BL, symbol haven_dev_board:U10
- removed U14: MX25R6435FBFIL0, haven_footprints:WLCSP-22_MX25R6435FBFIL0, symbol haven_dev_board:U14
- removed U6: BQ27220YZFR, haven_footprints:DSBGA-9_L1.7-W1.6-R3-C3-P0.50-BL, symbol haven_dev_board:U6
- removed U9: AP22916BCA4-7, haven_footprints:X1-WLB0808-4_L0.8-W0.8-P0.40-TL, symbol haven_dev_board:U9
- J1: now not fitted; now left out of the parts list
- R21: value 10mΩ, 1% -> 0R
